File: enigma_hut/switch_board.kicad_sch (KiCad schematic)
At the start: 27 parts, among them J1 Conn_02x08_Counter_Clockwise, SW1 SW_Push, SW10 SW_Push, SW11 SW_Push, SW12 SW_Push, SW13 SW_Push, SW14 SW_Push, SW15 SW_Push, SW16 SW_Push, SW17 SW_Push, SW18 SW_Push, SW19 SW_Push, SW2 SW_Push, SW20 SW_Push, SW21 SW_Push, SW22 SW_Push, SW23 SW_Push, SW24 SW_Push, SW25 SW_Push, SW26 SW_Push, SW3 SW_Push, SW4 SW_Push, SW5 SW_Push, SW6 SW_Push, SW7 SW_Push, SW8 SW_Push, SW9 SW_Push

Commit message: Update
Connections:
- net 11910 renamed c4
- net c4: now also SW14.2; no longer SW11.2
- net 141213 renamed c5
- net c5: now also SW17.2; no longer SW14.2
- net 171516 renamed c6
- net c6: now also SW20.2; no longer SW17.2
- net 201819 renamed c7
- net c7: now also SW23.2; no longer SW20.2
- net 21 renamed c1
- net c1: now also SW5.2
- net 232122 renamed c8
- net c8: now also SW26.2; no longer SW23.2
- net 262425 renamed c9
- net c9: no longer SW26.2
- net 534 renamed c2
- net c2: now also SW8.2; no longer SW5.2
- net 867 renamed c3
- net c3: now also SW11.2; no longer SW8.2
