File: Schematics/cont_board/cont_board.kicad_pcb (KiCad board)
At the start: 2 copper layers, 238 x 67 mm, 45 parts, among them IC1 LM2931AZ-5.0_TO92, J1 Conn_01x04, J2 Conn_01x04, J3 Conn_01x04, J4 Conn_01x04, Q1 BD438, Q2 BD438, Q3 BD438, SW1 SW_SPDT, U1 LM317_TO-220, U2 MCP23017_SP, U3 ULN2803A, U4 MCP23017_SP, U5 ULN2803A

Commit message: Cont-board rev1.1 done and sent to manufacturing
Parts:
- F1: value 1A -> 1A Slow Blow
- J1, J2, J3, J4: footprint Connector_PinHeader_2.54mm:PinHeader_1x04_P2.54mm_Vertical -> user_global_footprints:PinHeader_1x04_P2.54mm_Vertical_SLIM
- moved H1 134.2 mm to (30.0, 122.5)
- moved H2 134.2 mm to (30.0, 64.5)
- moved H3 134.2 mm to (258.0, 64.5)
- moved H4 134.2 mm to (117.5, 83.5)
- moved H5 134.2 mm to (258.0, 122.5)
- moved H6 134.2 mm to (173.5, 105.5)
- moved PL3 19.0 mm to (257.7, 82.1)
- moved JP4 18.6 mm to (182.2, 109.9)
- moved JP5 18.6 mm to (182.2, 113.0)
- moved JP6 18.6 mm to (182.2, 116.2)
- moved J4 17.2 mm to (166.4, 69.8)
- moved J1 17.2 mm to (158.8, 69.8)
- moved J3 17.2 mm to (163.8, 69.8)
- moved J2 17.2 mm to (161.3, 69.8)
- moved U3 16.6 mm to (196.2, 66.0)
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Connections:
- net Net-(JP1-C) renamed /s_a2
- net Net-(JP2-C) renamed /s_a1
- net Net-(JP3-C) renamed /s_a0
- net Net-(JP4-C) renamed /lamp_drive/l_a2
- net Net-(JP5-C) renamed /lamp_drive/l_a1
- net Net-(JP6-C) renamed /lamp_drive/l_a0
Routing:
- net +5V: track 285.0 -> 312.4 mm
- net +12VA: track 196.7 -> 212.0 mm
- net GND: track 11.3 -> 26.5 mm, vias 5 -> 6
- net CAM1_POS: track 89.2 -> 97.4 mm
- net CAM2_POS: track 86.9 -> 94.7 mm
- net SDA: track 175.1 -> 181.8 mm
- net SCL: track 175.5 -> 181.5 mm
- net /lamp_drive/c9: track 61.7 -> 66.0 mm
- net /lamp_drive/c3: track 58.3 -> 62.6 mm
- net /lamp_drive/l_a2: track 13.6 -> 17.8 mm
- net /lamp_drive/c2: track 52.9 -> 56.8 mm
- net /lamp_drive/c8: track 61.0 -> 64.4 mm
- net /lamp_drive/c7: track 61.0 -> 64.4 mm
- net /lamp_drive/c5: track 61.4 -> 64.8 mm
- net /lamp_drive/c6: track 61.0 -> 64.4 mm
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Other:
- board text added: "-"
- board text added: "04/12/2023 - last rev. 06/12/2023"
- board text added: "0V"
- board text added: "5V<-"
- board text added: "B+"
- board text added: "C1+"
- board text added: "C2+"
- board text added: "CUED | LZB - Enigma Control Board v1.1"
- board text added: "D13"
- board text added: "I2C Breakouts"
- board text added: "Lamp Board Conn."
- board text added: "Switch Board Conn."
- board text added: "TEST <-"
- board text added: "https://github.com/lbligh/enigma-iib-lzb23"
- board text removed: "03/12/2023"
- board text removed: "5V"
- board text removed: "CUED | LZB - Enigma Control Board v1.0"
- board text removed: "TEST"
