File: Schematics/lmp_board/lmp_board.kicad_pcb (KiCad board)
At the start: 2 copper layers, 238 x 67 mm, 63 parts, among them J1 Conn_02x08_Odd_Even

Commit message: Lamp Board Work and drl2dxf
Parts:
- D1, D10, D11, D12, D13, D14, D15, D16, D17, D18, D19, D2, D20, D21, D22, D23, D24, D25, D26, D27, D28, D3, D4, D5, D6, D7, D8, D9: footprint Diode_THT:D_DO-41_SOD81_P10.16mm_Horizontal -> user_global_footprints:D_DO-41_SOD81_P10.16mm_Horizontal_no_cathode
- moved D9 15.5 mm to (252.0, 63.0), turned to 180 degrees
- moved D28 7.17 mm to (244.0, 122.5), turned to 180 degrees
- moved LA10 4.47 mm to (253.5, 92.5)
- moved D1 2.00 mm to (60.0, 65.0)
- moved D11 2.00 mm to (44.0, 87.0)
- moved D12 2.00 mm to (68.0, 87.0)
- moved D13 2.00 mm to (92.0, 87.0)
- moved D14 2.00 mm to (116.0, 87.0)
- moved D15 2.00 mm to (140.0, 87.0)
- moved D16 2.00 mm to (164.0, 87.0)
- moved D17 2.00 mm to (188.0, 87.0)
- moved D18 2.00 mm to (212.0, 87.0)
- moved D19 2.00 mm to (236.0, 87.0)
- moved D2 2.00 mm to (84.0, 65.0)
- moved D20 2.00 mm to (52.0, 120.0)
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Routing:
- net /row2: track 0.00 -> 319.5 mm, vias 0 -> 1
- net /col1: track 0.00 -> 278.9 mm
- net /col2: track 0.00 -> 253.9 mm
- net /row1: track 0.00 -> 240.3 mm
- net /col3: track 0.00 -> 232.5 mm
- net /row3: track 0.00 -> 220.0 mm
- net /col4: track 0.00 -> 211.0 mm
- net /col5: track 0.00 -> 196.2 mm
- net /col6: track 0.00 -> 168.9 mm
- net /col7: track 0.00 -> 134.7 mm, vias 0 -> 1
- net /col8: track 0.00 -> 128.3 mm
- net /col9: track 0.00 -> 76.3 mm
- net /LT-: track 0.00 -> 39.3 mm, vias 0 -> 1
- net /LT+: track 0.00 -> 35.1 mm
- net /LT: track 0.00 -> 15.7 mm
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Other:
- board text added: "06/12/2023 - last rev. 09/12/2023"
- board text removed: "06/12/2023 - last rev. 06/12/2023"
- board text removed: "Switch Board Conn."
