File: Schematics/lmp_board/lmp_board.kicad_sch (KiCad schematic)
At the start: 57 parts, among them J2 Conn_02x08_Counter_Clockwise

Commit message: Lamp Board Schematic started
Parts:
- removed D2, D27: D, symbol Device:D
- removed J2: Conn_02x08_Counter_Clockwise, symbol Connector_Generic:Conn_02x08_Counter_Clockwise
- removed LA23, LA27: Lamp, symbol Device:Lamp
- added D18, D19: D, Diode_THT:D_DO-41_SOD81_P10.16mm_Horizontal, symbol Device:D
- added H1, H2, H3, H4, H5, H6: MountingHole_Pad, MountingHole:MountingHole_3.2mm_M3_Pad_Via, symbol Mechanical:MountingHole
- added J1: Conn_02x08_Odd_Even, Connector_PinHeader_2.54mm:PinHeader_2x08_P2.54mm_Vertical, symbol Connector_Generic:Conn_02x08_Odd_Even
- added LA18: J, user_global_footprints:Bulb_Holder_Temp, symbol Device:Lamp
- added LA19: K, user_global_footprints:Bulb_Holder_Temp, symbol Device:Lamp
- D1, D14: footprint (none) -> Diode_THT:D_DO-41_SOD81_P10.16mm_Horizontal
- D10: renamed from D28; footprint (none) -> Diode_THT:D_DO-41_SOD81_P10.16mm_Horizontal
- D11: renamed from D23; footprint (none) -> Diode_THT:D_DO-41_SOD81_P10.16mm_Horizontal
- D12: renamed from D20; footprint (none) -> Diode_THT:D_DO-41_SOD81_P10.16mm_Horizontal
- D13: renamed from D17; footprint (none) -> Diode_THT:D_DO-41_SOD81_P10.16mm_Horizontal
- D15: renamed from D11; footprint (none) -> Diode_THT:D_DO-41_SOD81_P10.16mm_Horizontal
- D16: renamed from D8; footprint (none) -> Diode_THT:D_DO-41_SOD81_P10.16mm_Horizontal
- D17: renamed from D5; footprint (none) -> Diode_THT:D_DO-41_SOD81_P10.16mm_Horizontal
- D2: renamed from D4; footprint (none) -> Diode_THT:D_DO-41_SOD81_P10.16mm_Horizontal
- D20: renamed from D3; footprint (none) -> Diode_THT:D_DO-41_SOD81_P10.16mm_Horizontal
- D21: renamed from D6; footprint (none) -> Diode_THT:D_DO-41_SOD81_P10.16mm_Horizontal
- D22: renamed from D9; footprint (none) -> Diode_THT:D_DO-41_SOD81_P10.16mm_Horizontal
- D23: renamed from D12; footprint (none) -> Diode_THT:D_DO-41_SOD81_P10.16mm_Horizontal
- D24: renamed from D15; footprint (none) -> Diode_THT:D_DO-41_SOD81_P10.16mm_Horizontal
- D25: renamed from D18; footprint (none) -> Diode_THT:D_DO-41_SOD81_P10.16mm_Horizontal
- D26: renamed from D21; footprint (none) -> Diode_THT:D_DO-41_SOD81_P10.16mm_Horizontal
- D27: renamed from D24; footprint (none) -> Diode_THT:D_DO-41_SOD81_P10.16mm_Horizontal
- D28: renamed from D26; footprint (none) -> Diode_THT:D_DO-41_SOD81_P10.16mm_Horizontal
- D3: renamed from D7; footprint (none) -> Diode_THT:D_DO-41_SOD81_P10.16mm_Horizontal
- D4: renamed from D10; footprint (none) -> Diode_THT:D_DO-41_SOD81_P10.16mm_Horizontal
- D5: renamed from D13; footprint (none) -> Diode_THT:D_DO-41_SOD81_P10.16mm_Horizontal
- D6: renamed from D16; footprint (none) -> Diode_THT:D_DO-41_SOD81_P10.16mm_Horizontal
- D7: renamed from D19; footprint (none) -> Diode_THT:D_DO-41_SOD81_P10.16mm_Horizontal
- D8: renamed from D22; footprint (none) -> Diode_THT:D_DO-41_SOD81_P10.16mm_Horizontal
- D9: renamed from D25; footprint (none) -> Diode_THT:D_DO-41_SOD81_P10.16mm_Horizontal
- LA1: value Lamp -> Q; footprint (none) -> user_global_footprints:Bulb_Holder_Temp
- LA10: renamed from LA28; value Lamp -> LT; footprint (none) -> user_global_footprints:Bulb_Holder_Temp
- LA11: renamed from LA2; value Lamp -> ST; footprint (none) -> user_global_footprints:Bulb_Holder_Temp
- LA12: renamed from LA5; value Lamp -> A; footprint (none) -> user_global_footprints:Bulb_Holder_Temp
- LA13: renamed from LA8; value Lamp -> S; footprint (none) -> user_global_footprints:Bulb_Holder_Temp
- LA14: renamed from LA11; value Lamp -> D; footprint (none) -> user_global_footprints:Bulb_Holder_Temp
- LA15: renamed from LA14; value Lamp -> F; footprint (none) -> user_global_footprints:Bulb_Holder_Temp
- LA16: renamed from LA17; value Lamp -> G; footprint (none) -> user_global_footprints:Bulb_Holder_Temp
- LA17: renamed from LA20; value Lamp -> H; footprint (none) -> user_global_footprints:Bulb_Holder_Temp
- LA2: renamed from LA4; value Lamp -> W; footprint (none) -> user_global_footprints:Bulb_Holder_Temp
- LA20: renamed from LA3; value Lamp -> P; footprint (none) -> user_global_footprints:Bulb_Holder_Temp
- LA21: renamed from LA6; value Lamp -> Y; footprint (none) -> user_global_footprints:Bulb_Holder_Temp
- LA22: renamed from LA9; value Lamp -> X; footprint (none) -> user_global_footprints:Bulb_Holder_Temp
- LA23: renamed from LA12; value Lamp -> C; footprint (none) -> user_global_footprints:Bulb_Holder_Temp
- LA24: renamed from LA15; value Lamp -> V; footprint (none) -> user_global_footprints:Bulb_Holder_Temp
- LA25: renamed from LA18; value Lamp -> B; footprint (none) -> user_global_footprints:Bulb_Holder_Temp
- LA26: renamed from LA21; value Lamp -> N; footprint (none) -> user_global_footprints:Bulb_Holder_Temp
- LA27: renamed from LA24; value Lamp -> M; footprint (none) -> user_global_footprints:Bulb_Holder_Temp
- LA28: renamed from LA26; value Lamp -> L; footprint (none) -> user_global_footprints:Bulb_Holder_Temp
- LA3: renamed from LA7; value Lamp -> E; footprint (none) -> user_global_footprints:Bulb_Holder_Temp
- LA4: renamed from LA10; value Lamp -> R; footprint (none) -> user_global_footprints:Bulb_Holder_Temp
- LA5: renamed from LA13; value Lamp -> T; footprint (none) -> user_global_footprints:Bulb_Holder_Temp
- LA6: renamed from LA16; value Lamp -> Z; footprint (none) -> user_global_footprints:Bulb_Holder_Temp
- LA7: renamed from LA19; value Lamp -> U; footprint (none) -> user_global_footprints:Bulb_Holder_Temp
- LA8: renamed from LA22; value Lamp -> I; footprint (none) -> user_global_footprints:Bulb_Holder_Temp
- LA9: renamed from LA25; value Lamp -> O; footprint (none) -> user_global_footprints:Bulb_Holder_Temp
Connections:
- net col1: now also J1.15 (Pin_15)
- net col2: now also J1.13 (Pin_13)
- net col3: now also J1.11 (Pin_11)
- net col4: now also J1.9 (Pin_9)
- net col5: now also J1.7 (Pin_7)
- net col6: now also J1.5 (Pin_5)
- net col7: now also J1.3 (Pin_3)
- net col8: now also J1.1 (Pin_1), LA18.2 (+)
- net col9: now also J1.10 (Pin_10), LA19.2 (+)
- net row1: now also J1.16 (Pin_16)
- net row2: now also D18.2 (A), D19.2 (A), J1.14 (Pin_14)
- net row3: now also J1.12 (Pin_12)
- net C: now reaches D23.1 (K), LA23.1 (-)
- net N: now reaches D26.1 (K), LA26.1 (-)
- net L: now reaches D28.1 (K), LA28.1 (-)
- net T: now reaches D5.1 (K), LA5.1 (-)
- net LT-: now reaches LA10.2 (+)
- net LT-: now also J1.4 (Pin_4)
- net I: now reaches D8.1 (K), LA8.1 (-)
- net S: now reaches D13.1 (K), LA13.1 (-)
- net H: now reaches D17.1 (K), LA17.1 (-)
- net M: now reaches D27.1 (K), LA27.1 (-)
- net ST: now reaches D11.1 (K), LA11.1 (-)
- net G: now reaches D16.1 (K), LA16.1 (-)
- net Y: now reaches D21.1 (K), LA21.1 (-)
- net B: now reaches D25.1 (K), LA25.1 (-)
- net D: now reaches D14.1 (K), LA14.1 (-)
- net E: now reaches D3.1 (K), LA3.1 (-)
- net V: now reaches D24.1 (K), LA24.1 (-)
- net O: now reaches D9.1 (K), LA9.1 (-)
- net F: now reaches D15.1 (K), LA15.1 (-)
- net Z: now reaches D6.1 (K), LA6.1 (-)
- net X: now reaches D22.1 (K), LA22.1 (-)
- net A: now reaches D12.1 (K), LA12.1 (-)
- net LT: now reaches D10.1 (K), LA10.1 (-)
- net U: now reaches D7.1 (K), LA7.1 (-)
- net LT+: now reaches D10.2 (A)
- net LT+: now also J1.2 (Pin_2)
- net R: now reaches D4.1 (K), LA4.1 (-)
- net W: now reaches D2.1 (K), LA2.1 (-)
- net P: now reaches D20.1 (K), LA20.1 (-)
- net Q: now reaches D1.1 (K), LA1.1 (-)
- new net J: D18.1 (K), LA18.1 (-)
- new net K: D19.1 (K), LA19.1 (-)
Other:
- moved on the sheet: D10, LA11, LA12, LA13, LA14, LA15, LA16, LA17

Commit message: Lamp Board Work and drl2dxf
Parts:
- D1, D10, D11, D12, D13, D14, D15, D16, D17, D18, D19, D2, D20, D21, D22, D23, D24, D25, D26, D27, D28, D3, D4, D5, D6, D7, D8, D9: footprint Diode_THT:D_DO-41_SOD81_P10.16mm_Horizontal -> user_global_footprints:D_DO-41_SOD81_P10.16mm_Horizontal_no_cathode
Changed lines of the file:
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@@
       (effects (font (size 1.27 1.27)))
     )
-    (property "Footprint" "Diode_THT:D_DO-41_SOD81_P10.16mm_Horizontal" (at 166.37 151.13 0)
+    (property "Footprint" "user_global_footprints:D_DO-41_SOD81_P10.16mm_Horizontal_no_cathode" (at 166.37 151.13 0)
       (effects (font (size 1.27 1.27)) hide)
     )
@@
       (effects (font (size 1.27 1.27)))
     )
-    (property "Footprint" "Diode_THT:D_DO-41_SOD81_P10.16mm_Horizontal" (at 201.93 151.13 0)
+    (property "Footprint" "user_global_footprints:D_DO-41_SOD81_P10.16mm_Horizontal_no_cathode" (at 201.93 151.13 0)
       (effects (font (size 1.27 1.27)) hide)
     )
@@
       (effects (font (size 1.27 1.27)))
     )
-    (property "Footprint" "Diode_THT:D_DO-41_SOD81_P10.16mm_Horizontal" (at 130.81 41.91 0)
+    (property "Footprint" "user_global_footprints:D_DO-41_SOD81_P10.16mm_Horizontal_no_cathode" (at 130.81 41.91 0)
       (effects (font (size 1.27 1.27)) hide)
     )
@@
       (effects (font (size 1.27 1.27)) (justify left))
     )
-    (property "Footprint" "Diode_THT:D_DO-41_SOD81_P10.16mm_Horizontal" (at 167.64 90.17 0)
+    (property "Footprint" "user_global_footprints:D_DO-41_SOD81_P10.16mm_Horizontal_no_cathode" (at 167.64 90.17 0)
       (effects (font (size 1.27 1.27)) hide)
     )
@@
       (effects (font (size 1.27 1.27)))
     )
-    (property "Footprint" "Diode_THT:D_DO-41_SOD81_P10.16mm_Horizontal" (at 184.15 151.13 0)
+    (property "Footprint" "user_global_footprints:D_DO-41_SOD81_P10.16mm_Horizontal_no_cathode" (at 184.15 151.13 0)
       (effects (font (size 1.27 1.27)) hide)
     )
@@
       (effects (font (size 1.27 1.27)))
     )
-    (property "Footprint" "Diode_THT:D_DO-41_SOD81_P10.16mm_Horizontal" (at 148.59 151.13 0)
+    (property "Footprint" "user_global_footprints:D_DO-41_SOD81_P10.16mm_Horizontal_no_cathode" (at 148.59 151.13 0)
       (effects (font (size 1.27 1.27)) hide)
     )
@@
       (effects (font (size 1.27 1.27)) (justify left))
     )
-    (property "Footprint" "Diode_THT:D_DO-41_SOD81_P10.16mm_Horizontal" (at 114.3 90.17 0)
+    (property "Footprint" "user_global_footprints:D_DO-41_SOD81_P10.16mm_Horizontal_no_cathode" (at 114.3 90.17 0)
       (effects (font (size 1.27 1.27)) hide)
     )
@@
       (effects (font (size 1.27 1.27)))
     )
-    (property "Footprint" "Diode_THT:D_DO-41_SOD81_P10.16mm_Horizontal" (at 95.25 41.91 0)
+    (property "Footprint" "user_global_footprints:D_DO-41_SOD81_P10.16mm_Horizontal_no_cathode" (at 95.25 41.91 0)
       (effects (font (size 1.27 1.27)) hide)
     )
@@
       (effects (font (size 1.27 1.27)))
     )
-    (property "Footprint" "Diode_THT:D_DO-41_SOD81_P10.16mm_Horizontal" (at 184.15 41.91 0)
+    (property "Footprint" "user_global_footprints:D_DO-41_SOD81_P10.16mm_Horizontal_no_cathode" (at 184.15 41.91 0)
       (effects (font (size 1.27 1.27)) hide)
     )
@@
       (effects (font (size 1.27 1.27)))
     )
-    (property "Footprint" "Diode_THT:D_DO-41_SOD81_P10.16mm_Horizontal" (at 113.03 151.13 0)
+    (property "Footprint" "user_global_footprints:D_DO-41_SOD81_P10.16mm_Horizontal_no_cathode" (at 113.03 151.13 0)
       (effects (font (size 1.27 1.27)) hide)
     )
@@
       (effects (font (size 1.27 1.27)))
     )
-    (property "Footprint" "Diode_THT:D_DO-41_SOD81_P10.16mm_Horizontal" (at 130.81 151.13 0)
+    (property "Footprint" "user_global_footprints:D_DO-41_SOD81_P10.16mm_Horizontal_no_cathode" (at 130.81 151.13 0)
       (effects (font (size 1.27 1.27)) hide)
     )
@@
       (effects (font (size 1.27 1.27)) (justify left))
     )
-    (property "Footprint" "Diode_THT:D_DO-41_SOD81_P10.16mm_Horizontal" (at 185.42 90.17 0)
+    (property "Footprint" "user_global_footprints:D_DO-41_SOD81_P10.16mm_Horizontal_no_cathode" (at 185.42 90.17 0)
       (effects (font (size 1.27 1.27)) hide)
     )
@@
       (effects (font (size 1.27 1.27)) (justify left))
     )
-    (property "Footprint" "Diode_THT:D_DO-41_SOD81_P10.16mm_Horizontal" (at 132.08 90.17 0)
+    (property "Footprint" "user_global_footprints:D_DO-41_SOD81_P10.16mm_Horizontal_no_cathode" (at 132.08 90.17 0)
       (effects (font (size 1.27 1.27)) hide)
     )
@@
       (effects (font (size 1.27 1.27)))
     )
-    (property "Footprint" "Diode_THT:D_DO-41_SOD81_P10.16mm_Horizontal" (at 148.59 41.91 0)
+    (property "Footprint" "user_global_footprints:D_DO-41_SOD81_P10.16mm_Horizontal_no_cathode" (at 148.59 41.91 0)
       (effects (font (size 1.27 1.27)) hide)
     )
@@
       (effects (font (size 1.27 1.27)) (justify left))
     )
-    (property "Footprint" "Diode_THT:D_DO-41_SOD81_P10.16mm_Horizontal" (at 78.74 90.17 0)
+    (property "Footprint" "user_global_footprints:D_DO-41_SOD81_P10.16mm_Horizontal_no_cathode" (at 78.74 90.17 0)
       (effects (font (size 1.27 1.27)) hide)
     )
@@
       (effects (font (size 1.27 1.27)) (justify left))
     )
-    (property "Footprint" "Diode_THT:D_DO-41_SOD81_P10.16mm_Horizontal" (at 203.2 90.17 0)
+    (property "Footprint" "user_global_footprints:D_DO-41_SOD81_P10.16mm_Horizontal_no_cathode" (at 203.2 90.17 0)
       (effects (font (size 1.27 1.27)) hide)
     )
@@
       (effects (font (size 1.27 1.27)))
     )
-    (property "Footprint" "Diode_THT:D_DO-41_SOD81_P10.16mm_Horizontal" (at 77.47 151.13 0)
+    (property "Footprint" "user_global_footprints:D_DO-41_SOD81_P10.16mm_Horizontal_no_cathode" (at 77.47 151.13 0)
       (effects (font (size 1.27 1.27)) hide)
     )
@@
       (effects (font (size 1.27 1.27)))
     )
-    (property "Footprint" "Diode_THT:D_DO-41_SOD81_P10.16mm_Horizontal" (at 95.25 151.13 0)
+    (property "Footprint" "user_global_footprints:D_DO-41_SOD81_P10.16mm_Horizontal_no_cathode" (at 95.25 151.13 0)
       (effects (font (size 1.27 1.27)) hide)
     )
@@
       (effects (font (size 1.27 1.27)))
     )
-    (property "Footprint" "Diode_THT:D_DO-41_SOD81_P10.16mm_Horizontal" (at 166.37 41.91 0)
+    (property "Footprint" "user_global_footprints:D_DO-41_SOD81_P10.16mm_Horizontal_no_cathode" (at 166.37 41.91 0)
       (effects (font (size 1.27 1.27)) hide)
     )
@@
       (effects (font (size 1.27 1.27)) (justify left))
     )
-    (property "Footprint" "Diode_THT:D_DO-41_SOD81_P10.16mm_Horizontal" (at 149.86 90.17 0)
+    (property "Footprint" "user_global_footprints:D_DO-41_SOD81_P10.16mm_Horizontal_no_cathode" (at 149.86 90.17 0)
       (effects (font (size 1.27 1.27)) hide)
     )
@@
       (effects (font (size 1.27 1.27)))
     )
-    (property "Footprint" "Diode_THT:D_DO-41_SOD81_P10.16mm_Horizontal" (at 201.93 41.91 0)
+    (property "Footprint" "user_global_footprints:D_DO-41_SOD81_P10.16mm_Horizontal_no_cathode" (at 201.93 41.91 0)
       (effects (font (size 1.27 1.27)) hide)
     )
@@
       (effects (font (size 1.27 1.27)))
     )
-    (property "Footprint" "Diode_THT:D_DO-41_SOD81_P10.16mm_Horizontal" (at 77.47 41.91 0)
+    (property "Footprint" "user_global_footprints:D_DO-41_SOD81_P10.16mm_Horizontal_no_cathode" (at 77.47 41.91 0)
       (effects (font (size 1.27 1.27)) hide)
     )
@@
       (effects (font (size 1.27 1.27)))
     )
-    (property "Footprint" "Diode_THT:D_DO-41_SOD81_P10.16mm_Horizontal" (at 59.69 151.13 0)
+    (property "Footprint" "user_global_footprints:D_DO-41_SOD81_P10.16mm_Horizontal_no_cathode" (at 59.69 151.13 0)
       (effects (font (size 1.27 1.27)) hide)
     )
@@
       (effects (font (size 1.27 1.27)) (justify right))
     )
-    (property "Footprint" "Diode_THT:D_DO-41_SOD81_P10.16mm_Horizontal" (at 255.27 78.74 0)
+    (property "Footprint" "user_global_footprints:D_DO-41_SOD81_P10.16mm_Horizontal_no_cathode" (at 255.27 78.74 0)
       (effects (font (size 1.27 1.27)) hide)
     )
@@
       (effects (font (size 1.27 1.27)) (justify left))
     )
-    (property "Footprint" "Diode_THT:D_DO-41_SOD81_P10.16mm_Horizontal" (at 60.96 90.17 0)
+    (property "Footprint" "user_global_footprints:D_DO-41_SOD81_P10.16mm_Horizontal_no_cathode" (at 60.96 90.17 0)
       (effects (font (size 1.27 1.27)) hide)
     )
@@
       (effects (font (size 1.27 1.27)))
     )
-    (property "Footprint" "Diode_THT:D_DO-41_SOD81_P10.16mm_Horizontal" (at 113.03 41.91 0)
+    (property "Footprint" "user_global_footprints:D_DO-41_SOD81_P10.16mm_Horizontal_no_cathode" (at 113.03 41.91 0)
       (effects (font (size 1.27 1.27)) hide)
     )
@@
       (effects (font (size 1.27 1.27)) (justify left))
     )
-    (property "Footprint" "Diode_THT:D_DO-41_SOD81_P10.16mm_Horizontal" (at 96.52 90.17 0)
+    (property "Footprint" "user_global_footprints:D_DO-41_SOD81_P10.16mm_Horizontal_no_cathode" (at 96.52 90.17 0)
       (effects (font (size 1.27 1.27)) hide)
     )
@@
       (effects (font (size 1.27 1.27)))
     )
-    (property "Footprint" "Diode_THT:D_DO-41_SOD81_P10.16mm_Horizontal" (at 59.69 41.91 0)
-      (effects (font (size 1.27 1.27)) hide)
-    )
+    (property "Footprint" "user_global_footprints:D_DO-41_SOD81_P10.16mm_Horizontal_no_cathode" (at 59.69 41.91 0)
+      (effects (font (size 1.27 1.27)) hide)
+    )
